Commit message: tried running moveit but moveit setup assistant throwing errors

File: rover_ws/src/rover_description/urdf/rover.urdf.xacro (robot description, xacro)
@@ -27,10 +27,8 @@
   <xacro:property name="mid_x" value="0.0"/>
   <xacro:property name="rear_x" value="-0.3"/>
-  <!-- Arm link lengths (meters) — HARDWARE UPGRADE: measure real arm -->
-  <xacro:property name="arm_base_height" value="0.1"/>
-  <xacro:property name="upper_arm_length" value="0.3"/>
-  <xacro:property name="forearm_length" value="0.25"/>
-  <xacro:property name="wrist_length" value="0.1"/>
-  <xacro:property name="gripper_length" value="0.08"/>
+  <!-- Arm link lengths (meters) — matches arm.urdf reference design -->
+  <xacro:property name="arm_base_height" value="0.05"/>
+  <xacro:property name="upper_arm_length" value="0.5"/>
+  <xacro:property name="forearm_length" value="0.5"/>
   <!-- ==================== MACROS ==================== -->
   <!-- Inertia for a box -->
@@ -98,15 +96,16 @@
   <xacro:wheel name="right_rear_wheel"  x="${rear_x}"  y="${-wheel_separation/2}"/>
   <!-- ==================== ARM ==================== -->
+  <!-- Base plate (flat cylinder, matches arm.urdf base_link) -->
   <link name="arm_base_link">
     <visual>
-      <geometry><cylinder radius="0.04" length="${arm_base_height}"/></geometry>
-      <origin xyz="0 0 ${arm_base_height/2}"/>
+      <origin xyz="0 0 ${arm_base_height/2}" rpy="0 0 0"/>
+      <geometry><cylinder radius="0.1" length="${arm_base_height}"/></geometry>
       <material name="grey"><color rgba="0.5 0.5 0.5 1"/></material>
     </visual>
     <collision>
-      <geometry><cylinder radius="0.04" length="${arm_base_height}"/></geometry>
-      <origin xyz="0 0 ${arm_base_height/2}"/>
-    </collision>
-    <xacro:cylinder_inertia mass="0.5" r="0.04" l="${arm_base_height}"/>
+      <origin xyz="0 0 ${arm_base_height/2}" rpy="0 0 0"/>
+      <geometry><cylinder radius="0.1" length="${arm_base_height}"/></geometry>
+    </collision>
+    <xacro:cylinder_inertia mass="1.0" r="0.1" l="${arm_base_height}"/>
   </link>
   <joint name="arm_base_joint" type="fixed">
@@ -115,99 +114,81 @@
     <origin xyz="0.1 0 ${chassis_height}"/>
   </joint>
-  <!-- Joint 1: base_yaw (revolute, Z-axis) -->
+  <!-- Rotating base block (matches arm.urdf base_rot) -->
   <link name="shoulder_link">
     <visual>
-      <geometry><box size="0.06 0.06 0.08"/></geometry>
-      <origin xyz="0 0 0.04"/>
+      <origin xyz="0 0 0.035" rpy="0 0 0"/>
+      <geometry><box size="0.1 0.1 0.07"/></geometry>
       <material name="orange"><color rgba="0.8 0.4 0.1 1"/></material>
     </visual>
-    <xacro:box_inertia mass="0.3" x="0.06" y="0.06" z="0.08"/>
+    <collision>
+      <origin xyz="0 0 0.035" rpy="0 0 0"/>
+      <geometry><box size="0.1 0.1 0.07"/></geometry>
+    </collision>
+    <xacro:box_inertia mass="0.5" x="0.1" y="0.1" z="0.07"/>
   </link>
   <joint name="base_yaw" type="revolute">
     <parent link="arm_base_link"/>
     <child link="shoulder_link"/>
-    <origin xyz="0 0 ${arm_base_height}"/>
-    <axis xyz="0 0 1"/>
-    <limit lower="-3.14" upper="3.14" velocity="10.0" effort="1.2"/>
-  </joint>
-  <!-- Joint 2: shoulder_pitch (revolute, Y-axis) -->
+    <origin xyz="0 0 ${arm_base_height}" rpy="0 0 0"/>
+    <axis xyz="0 0 -1"/>
+    <limit lower="-6.28" upper="6.28" effort="10.0" velocity="1.0"/>
+  </joint>
+  <!-- Upper arm (matches arm.urdf arm1) -->
   <link name="upper_arm_link">
     <visual>
-      <geometry><box size="0.04 0.04 ${upper_arm_length}"/></geometry>
-      <origin xyz="0 0 ${upper_arm_length/2}"/>
+      <origin xyz="0 0 ${upper_arm_length/2}" rpy="0 0 0"/>
+      <geometry><cylinder length="${upper_arm_length}" radius="0.02"/></geometry>
       <material name="orange"/>
     </visual>
-    <xacro:box_inertia mass="1.0" x="0.04" y="0.04" z="${upper_arm_length}"/>
+    <collision>
+      <origin xyz="0 0 ${upper_arm_length/2}" rpy="0 0 0"/>
+      <geometry><cylinder length="${upper_arm_length}" radius="0.02"/></geometry>
+    </collision>
+    <xacro:cylinder_inertia mass="0.3" r="0.02" l="${upper_arm_length}"/>
   </link>
   <joint name="shoulder_pitch" type="revolute">
     <parent link="shoulder_link"/>
     <child link="upper_arm_link"/>
-    <origin xyz="0 0 0.08"/>
-    <axis xyz="0 1 0"/>
-    <limit lower="-1.57" upper="1.57" velocity="5.0" effort="12.0"/>
-  </joint>
-  <!-- Joint 3: elbow_pitch (revolute, Y-axis) -->
+    <origin xyz="0 0 0.07" rpy="0 0 0"/>
+    <axis xyz="1 0 0"/>
+    <limit lower="-1.57" upper="1.57" effort="10.0" velocity="1.0"/>
+  </joint>
+  <!-- Forearm (matches arm.urdf arm2) -->
   <link name="forearm_link">
     <visual>
-      <geometry><box size="0.035 0.035 ${forearm_length}"/></geometry>
-      <origin xyz="0 0 ${forearm_length/2}"/>
+      <origin xyz="0 0 ${forearm_length/2}" rpy="0 0 0"/>
+      <geometry><cylinder length="${forearm_length}" radius="0.02"/></geometry>
       <material name="orange"/>
     </visual>
-    <xacro:box_inertia mass="0.6" x="0.035" y="0.035" z="${forearm_length}"/>
+    <collision>
+      <origin xyz="0 0 ${forearm_length/2}" rpy="0 0 0"/>
+      <geometry><cylinder length="${forearm_length}" radius="0.02"/></geometry>
+    </collision>
+    <xacro:cylinder_inertia mass="0.3" r="0.02" l="${forearm_length}"/>
   </link>
   <joint name="elbow_pitch" type="revolute">
     <parent link="upper_arm_link"/>
     <child link="forearm_link"/>
-    <origin xyz="0 0 ${upper_arm_length}"/>
-    <axis xyz="0 1 0"/>
-    <limit lower="-2.35" upper="2.35" velocity="5.0" effort="12.0"/>
-  </joint>
-  <!-- Joint 4: wrist_roll (revolute, Z-axis) -->
-  <link name="wrist_link">
-    <visual>
-      <geometry><cylinder radius="0.025" length="${wrist_length}"/></geometry>
-      <origin xyz="0 0 ${wrist_length/2}"/>
+    <origin xyz="0.08 0 ${upper_arm_length}" rpy="0 0 0"/>
+    <axis xyz="1 0 0"/>
+    <limit lower="-3.14" upper="3.14" effort="10.0" velocity="1.0"/>
+  </joint>
+  <!-- End effector (matches arm.urdf ee_link) -->
+  <link name="gripper_link">
+    <visual>
+      <origin xyz="0 0 0.025" rpy="0 0 0"/>
+      <geometry><box size="0.1 0.1 0.05"/></geometry>
       <material name="grey"/>
     </visual>
-    <xacro:cylinder_inertia mass="0.2" r="0.025" l="${wrist_length}"/>
-  </link>
-  <joint name="wrist_roll" type="revolute">
+    <collision>
+      <origin xyz="0 0 0.025" rpy="0 0 0"/>
+      <geometry><box size="0.1 0.1 0.05"/></geometry>
+    </collision>
+    <xacro:box_inertia mass="0.2" x="0.1" y="0.1" z="0.05"/>
+  </link>
+  <joint name="gripper" type="fixed">
     <parent link="forearm_link"/>
-    <child link="wrist_link"/>
-    <origin xyz="0 0 ${forearm_length}"/>
-    <axis xyz="0 0 1"/>
-    <limit lower="-3.14" upper="3.14" velocity="8.0" effort="3.6"/>
-  </joint>
-  <!-- Joint 5: wrist_pitch (revolute, Y-axis) -->
-  <link name="wrist_pitch_link">
-    <visual>
-      <geometry><box size="0.03 0.03 0.04"/></geometry>
-      <origin xyz="0 0 0.02"/>
-      <material name="grey"/>
-    </visual>
-    <xacro:box_inertia mass="0.1" x="0.03" y="0.03" z="0.04"/>
-  </link>
-  <joint name="wrist_pitch" type="revolute">
-    <parent link="wrist_link"/>
-    <child link="wrist_pitch_link"/>
-    <origin xyz="0 0 ${wrist_length}"/>
-    <axis xyz="0 1 0"/>
-    <limit lower="-1.57" upper="1.57" velocity="8.0" effort="3.6"/>
-  </joint>
-  <!-- Joint 6: gripper (revolute, Z-axis) -->
-  <link name="gripper_link">
-    <visual>
-      <geometry><box size="0.06 0.08 ${gripper_length}"/></geometry>
-      <origin xyz="0 0 ${gripper_length/2}"/>
-      <material name="grey"/>
-    </visual>
-    <xacro:box_inertia mass="0.15" x="0.06" y="0.08" z="${gripper_length}"/>
-  </link>
-  <joint name="gripper" type="revolute">
-    <parent link="wrist_pitch_link"/>
     <child link="gripper_link"/>
-    <origin xyz="0 0 0.04"/>
-    <axis xyz="0 0 1"/>
-    <limit lower="0" upper="1.57" velocity="10.0" effort="1.2"/>
+    <origin xyz="0 0 ${forearm_length}" rpy="0 0 0"/>
   </joint>
   <!-- ==================== CAMERAS ==================== -->
